Commit message: Integrated LD19 Lidar Driver (ldrobot-lidar-ros2). Created launch file for the real robot (real_robot.launch.py)

File: description/lidar.xacro (robot description, xacro)
@@ -1,17 +1,20 @@
 <?xml version="1.0"?>
 <robot xmlns:xacro="http://www.ros.org/wiki/xacro" >
-    <joint name="laser_joint" type="fixed">
-        <parent link="chassis"/>
-        <child link="laser_frame"/>
-        <origin xyz="0.1 0 0.175" rpy="0 0 0" />
-    </joint>
-    <link name="laser_frame">
+    <!-- Lidar's base frame-->
+    <link name="ldlidar_base">
         <visual>
+            <origin xyz="0 0 0" rpy="0 0 0"/>
             <geometry>
                 <cylinder radius="0.05" length="0.04"/>
             </geometry>
             <material name="black"/>
+            <!-- <geometry>
+                <mesh filename="package://vacuum_bot/description/model/LD19.stl" scale="0.001 0.001 0.001" />
+            </geometry> -->
+            <material name="ldlidar_mat">
+                <color rgba="0.8 0.8 0.8 0.8"/>
+            </material>
         </visual>
-        <collision>
+        <!-- <collision>
             <geometry>
                 <cylinder radius="0.05" length="0.04"/>
@@ -20,7 +23,26 @@
         <xacro:inertial_cylinder mass="0.1" length="0.04" radius="0.05">
             <origin xyz="0 0 0" rpy="0 0 0"/>
-        </xacro:inertial_cylinder>
+        </xacro:inertial_cylinder> -->
     </link>
-    <gazebo reference="laser_frame">
+    <!-- Joint from robot to lidar -->
+    <joint name="ldlidar_mount_joint" type="fixed">
+        <parent link="chassis"/>
+        <child link="ldlidar_base"/>
+        <origin xyz="0.1 0 0.175" rpy="0 0 0" />
+    </joint>
+    <joint name="ldlidar_link_joint" type="fixed">
+        <parent link="ldlidar_base"/>
+        <child link="ldlidar_link"/>
+        <origin xyz="0 0 0.02745" rpy="0 0 0" />
+    </joint>
+    <link name="ldlidar_link">
+        <visual>
+            <geometry>
+                <sphere radius="0.01"/>
+            </geometry>
+            <material name="black"/>
+        </visual>
+    </link>
+    <gazebo reference="ldlidar_base">
         <material>Gazebo/Black</material>
         <sensor name="laser" type="gpu_lidar">
@@ -47,5 +69,5 @@
             </lidar>
             <topic>scan</topic>
-            <gz_frame_id>laser_frame</gz_frame_id>
+            <gz_frame_id>ldlidar_base</gz_frame_id>
         </sensor>
     </gazebo>
